Commit message: C/C++연결 테스트

File: snt_robot_description/xacro/SNTRobot.urdf.xacro (robot description, xacro)
@@ -16,5 +16,5 @@
     <color rgba="0.05 0.05 0.05 1.0"/>
   </material>
-  <material name="mat_orange">robot
+  <material name="mat_orange">
     <color rgba="1.0 0.45 0.0 1.0"/>
   </material>
